Commit message: Add changes

File: spincopter_description/urdf/firefly.xacro (robot description, xacro)
@@ -27,5 +27,6 @@
   <xacro:property name="mass_rotor" value="0.005" /> <!-- [kg] -->
   <xacro:property name="arm_length" value="0.215" /> <!-- [m] -->
-  <xacro:property name="rotor_offset_top" value="0.037" /> <!-- [m] -->
+  <xacro:property name="rotor_offset_top1" value="0.027" /> <!-- [m] -->
+  <xacro:property name="rotor_offset_top2" value="0.010" />
   <xacro:property name="radius_rotor" value="0.1" /> <!-- [m] -->
   <xacro:property name="motor_constant" value="8.54858e-06" /> <!-- [kg m/s^2] -->
@@ -38,4 +39,10 @@
   <xacro:property name="rotor_drag_coefficient" value="8.06428e-05" />
   <xacro:property name="rolling_moment_coefficient" value="0.000001" />
+  <xacro:property name="rotor_roll" value="1.047197" />
+  <xacro:property name="link_roll" value="1.57" />
+  <xacro:property name="link_mass" value="0.1" />
+  <xacro:property name="link_radius" value="0.01" />
+  <xacro:property name="link_offset_top" value="0.02" />
+  <xacro:property name="link_offset_base" value="0.1575" />
   <!-- Property Blocks -->
   <xacro:property name="body_inertia">
@@ -59,4 +66,28 @@
     <xacro:insert_block name="body_inertia" />
   </xacro:multirotor_base_macro>
+  <xacro:link_o
+    robot_namespace="${namespace}"
+    parent="${namespace}/base_link"
+    mass_link="${link_mass}"
+    radius_link="${link_radius}"
+    length_link="${arm_length}"
+    link_number="0"
+    color="Blue"
+    >
+    <origin xyz="${link_offset_base} 0 ${link_offset_top}" rpy="0 ${link_roll} 0" />
+    <xacro:insert_block name="rotor_inertia" />
+  </xacro:link_o>
+    <xacro:link_o
+    robot_namespace="${namespace}"
+    parent="${namespace}/base_link"
+    mass_link="${link_mass}"
+    radius_link="${link_radius}"
+    length_link="${arm_length}"
+    link_number="1"
+    color="Red"
+    >
+    <origin xyz="-${link_offset_base} 0 ${link_offset_top}" rpy="0 ${link_roll} 0" />
+    <xacro:insert_block name="rotor_inertia" />
+  </xacro:link_o>
   <!-- Instantiate rotors -->
   <xacro:vertical_rotor
@@ -76,12 +107,11 @@
     rolling_moment_coefficient="${rolling_moment_coefficient}"
     color="Red"
-    use_own_mesh="true"
+    use_own_mesh="False"
     mesh="">
-    <origin xyz="${cos30*arm_length} ${sin30*arm_length} ${rotor_offset_top}" rpy="0 0 0" />
+    <origin xyz="${arm_length} -${rotor_offset_top2} ${rotor_offset_top1}" rpy="${rotor_roll} 0 0" />
     <xacro:insert_block name="rotor_inertia" />
   </xacro:vertical_rotor>
-  <xacro:vertical_rotor
-    robot_namespace="${namespace}"
-    suffix="left"
+  <xacro:vertical_rotor robot_namespace="${namespace}"
+    suffix="back_right"
     direction="cw"
     motor_constant="${motor_constant}"
@@ -99,87 +129,5 @@
     use_own_mesh="false"
     mesh="">
-    <origin xyz="0 ${arm_length} ${rotor_offset_top}" rpy="0 0 0" />
-    <xacro:insert_block name="rotor_inertia" />
-  </xacro:vertical_rotor>
-  <xacro:vertical_rotor robot_namespace="${namespace}"
-    suffix="back_left"
-    direction="ccw"
-    motor_constant="${motor_constant}"
-    moment_constant="${moment_constant}"
-    parent="${namespace}/base_link"
-    mass_rotor="${mass_rotor}"
-    radius_rotor="${radius_rotor}"
-    time_constant_up="${time_constant_up}"
-    time_constant_down="${time_constant_down}"
-    max_rot_velocity="${max_rot_velocity}"
-    motor_number="2"
-    rotor_drag_coefficient="${rotor_drag_coefficient}"
-    rolling_moment_coefficient="${rolling_moment_coefficient}"
-    color="Blue"
-    use_own_mesh="false"
-    mesh="">
-    <origin xyz="-${cos30*arm_length} ${sin30*arm_length} ${rotor_offset_top}" rpy="0 0 0" />
-    <xacro:insert_block name="rotor_inertia" />
-  </xacro:vertical_rotor>
-  <xacro:vertical_rotor robot_namespace="${namespace}"
-    suffix="back_right"
-    direction="cw"
-    motor_constant="${motor_constant}"
-    moment_constant="${moment_constant}"
-    parent="${namespace}/base_link"
-    mass_rotor="${mass_rotor}"
-    radius_rotor="${radius_rotor}"
-    time_constant_up="${time_constant_up}"
-    time_constant_down="${time_constant_down}"
-    max_rot_velocity="${max_rot_velocity}"
-    motor_number="3"
-    rotor_drag_coefficient="${rotor_drag_coefficient}"
-    rolling_moment_coefficient="${rolling_moment_coefficient}"
-    color="Blue"
-    use_own_mesh="false"
-    mesh="">
-    <origin xyz="-${cos30*arm_length} -${sin30*arm_length} ${rotor_offset_top}" rpy="0 0 0" />
-    <xacro:insert_block name="rotor_inertia" />
-  </xacro:vertical_rotor>
-  <xacro:vertical_rotor
-    robot_namespace="${namespace}"
-    suffix="right"
-    direction="ccw"
-    motor_constant="${motor_constant}"
-    moment_constant="${moment_constant}"
-    parent="${namespace}/base_link"
-    mass_rotor="${mass_rotor}"
-    radius_rotor="${radius_rotor}"
-    time_constant_up="${time_constant_up}"
-    time_constant_down="${time_constant_down}"
-    max_rot_velocity="${max_rot_velocity}"
-    motor_number="4"
-    rotor_drag_coefficient="${rotor_drag_coefficient}"
-    rolling_moment_coefficient="${rolling_moment_coefficient}"
-    color="Blue"
-    use_own_mesh="false"
-    mesh="">
-    <origin xyz="0 -${arm_length} ${rotor_offset_top}" rpy="0 0 0" />
-    <xacro:insert_block name="rotor_inertia" />
-  </xacro:vertical_rotor>
-  <xacro:vertical_rotor
-    robot_namespace="${namespace}"
-    suffix="front_right"
-    direction="cw"
-    motor_constant="${motor_constant}"
-    moment_constant="${moment_constant}"
-    parent="${namespace}/base_link"
-    mass_rotor="${mass_rotor}"
-    radius_rotor="${radius_rotor}"
-    time_constant_up="${time_constant_up}"
-    time_constant_down="${time_constant_down}"
-    max_rot_velocity="${max_rot_velocity}"
-    motor_number="5"
-    rotor_drag_coefficient="${rotor_drag_coefficient}"
-    rolling_moment_coefficient="${rolling_moment_coefficient}"
-    color="Red"
-    use_own_mesh="false"
-    mesh="">
-    <origin xyz="${cos30*arm_length} -${sin30*arm_length} ${rotor_offset_top}" rpy="0 0 0" />
+    <origin xyz="-${arm_length} ${rotor_offset_top2} ${rotor_offset_top1}" rpy="-${rotor_roll} 0 0" />
     <xacro:insert_block name="rotor_inertia" />
   </xacro:vertical_rotor>

File: spincopter_description/urdf/firefly_base.xacro (robot description, xacro)
@@ -24,5 +24,5 @@
   <xacro:if value="$(arg enable_mavlink_interface)">
     <!-- Instantiate mavlink telemetry interface. -->
-    <xacro:default_mavlink_interface namespace="${namespace}" imu_sub_topic="imu" rotor_count="6" />
+    <xacro:default_mavlink_interface namespace="${namespace}" imu_sub_topic="imu" rotor_count="2" />
   </xacro:if>
   <!-- Mount an ADIS16448 IMU. -->

File: spincopter_description/urdf/multirotor_base.xacro (robot description, xacro)
@@ -73,4 +73,34 @@
     </gazebo>
   </xacro:macro>
+  <xacro:macro name="link_o"
+    params="robot_namespace parent mass_link radius_link length_link link_number color  *origin *inertia">
+    <joint name="${robot_namespace}/link_${link_number}_joint" type="fixed">
+      <xacro:insert_block name="origin" />
+      <axis xyz="0 0 1" />
+      <!-- TODO(ff): not currently set because it's not yet supported -->
+      <!-- <limit effort="2000" velocity="${max_rot_velocity}" /> -->
+      <parent link="${parent}" />
+      <child link="${robot_namespace}/link_${link_number}" />
+    </joint>
+    <link name="${robot_namespace}/link_${link_number}">
+      <inertial>
+        <mass value="${mass_link}" /> <!-- [kg] -->
+        <xacro:insert_block name="inertia" />
+      </inertial>
+      <visual>
+        <geometry>
+           <cylinder length="${length_link}" radius="${radius_link}"/>  <!-- [m] -->
+        </geometry>
+      </visual>
+      <collision>
+        <geometry>
+          <cylinder length="${length_link}" radius="${radius_link}" /> <!-- [m] -->
+        </geometry>
+      </collision>
+    </link>
+    <gazebo reference="${robot_namespace}/link_${link_number}">
+      <material>Gazebo/${color}</material>
+    </gazebo>
+  </xacro:macro>
   <!-- Rotor joint and link -->
   <xacro:macro name="vertical_rotor"
@@ -91,5 +121,6 @@
       <visual>
         <geometry>
-           <cylinder length="0.005" radius="${radius_rotor}"/>  <!-- [m] -->
+           <!--<cylinder length="0.005" radius="${radius_rotor}"/>  -->
+<!-- [m] -->
           <xacro:if value="${use_own_mesh}">
             <mesh filename="${mesh}"
