Commit message: Spincopter ready to fly

File: spincopter_description/urdf/rotor_wing_base.xacro (robot description, xacro)
@@ -23,4 +23,10 @@
       izz="${0.0833333 * mass * (x*x + y*y)}" />
   </xacro:macro>
+  <!-- Macro for the inertia of a cylinder -->
+  <xacro:macro name="cylinder_inertia" params="r h mass">
+    <inertia ixx="${0.0833333 * mass * (3*r*r + h*h)}" ixy="0.0" ixz="0.0"
+      iyy="${0.0833333 * mass * (3*r*r + h*h)}" iyz="0.0"
+      izz="${0.5 * mass * r * r}" />
+  </xacro:macro>
   <!-- Macro for the inertial properties of a box -->
   <xacro:macro name="box_inertial" params="x y z mass *origin">
@@ -163,3 +169,48 @@
     </gazebo>
   </xacro:macro>
+  <!-- Control surface joint and link -->
+  <xacro:macro name="control_surface"
+    params="robot_namespace surface_name parent mass_surface min_angle
+      max_angle color use_mesh_file mesh_file surface_length surface_width
+      surface_height *axis *joint_origin *link_origin *inertia">
+    <joint name="${robot_namespace}/${surface_name}_joint" type="revolute">
+      <xacro:insert_block name="joint_origin" />
+      <xacro:insert_block name="axis" />
+      <parent link="${parent}" />
+      <child link="${robot_namespace}/${surface_name}" />
+      <limit upper="${max_angle}" lower="${min_angle}" effort="0" velocity="0" />
+    </joint>
+    <link name="${robot_namespace}/${surface_name}">
+      <inertial>
+        <xacro:insert_block name="link_origin" />
+        <mass value="${mass_surface}" />
+        <xacro:insert_block name="inertia" />
+      </inertial>
+      <visual>
+        <xacro:insert_block name="link_origin" />
+        <geometry>
+          <xacro:if value="${use_mesh_file}">
+            <mesh filename="${mesh_file}" scale="1 1 1" />
+          </xacro:if>
+          <xacro:unless value="${use_mesh_file}">
+            <box size="${surface_length} ${surface_width} ${surface_height}" />
+          </xacro:unless>
+        </geometry>
+      </visual>
+      <collision>
+        <xacro:insert_block name="link_origin" />
+        <geometry>
+          <xacro:if value="${use_mesh_file}">
+            <mesh filename="${mesh_file}" scale="1 1 1" />
+          </xacro:if>
+          <xacro:unless value="${use_mesh_file}">
+            <box size="${surface_length} ${surface_width} ${surface_height}" />
+          </xacro:unless>
+        </geometry>
+      </collision>
+    </link>
+    <gazebo reference="${robot_namespace}/${surface_name}">
+      <material>Gazebo/${color}</material>
+    </gazebo>
+  </xacro:macro>
 </robot>

File: spincopter_description/urdf/spincopter.xacro (robot description, xacro)
@@ -20,5 +20,5 @@
   <xacro:property name="namespace" value="$(arg namespace)" />
   <xacro:property name="rotor_velocity_slowdown_sim" value="10" />
-  <xacro:property name="use_mesh_file" value="false" />
+  <xacro:property name="use_mesh_file" value="False" />
   <xacro:property name="mesh_file" value="package://rotors_description/meshes/firefly.dae" />
   <xacro:property name="mass" value="1.5" /> <!-- [kg] -->
@@ -27,6 +27,6 @@
   <xacro:property name="mass_rotor" value="0.005" /> <!-- [kg] -->
   <xacro:property name="arm_length" value="0.215" /> <!-- [m] -->
-  <xacro:property name="rotor_offset_top1" value="0.027" /> <!-- [m] -->
-  <xacro:property name="rotor_offset_top2" value="0.010" />
+  <xacro:property name="rotor_offset_top1" value="0.03" /> <!-- [m] -->
+  <xacro:property name="rotor_offset_top2" value="0.018" />
   <xacro:property name="radius_rotor" value="0.1" /> <!-- [m] -->
   <xacro:property name="motor_constant" value="8.54858e-06" /> <!-- [kg m/s^2] -->
@@ -45,14 +45,48 @@
   <xacro:property name="link_offset_top" value="0.02" />
   <xacro:property name="link_offset_base" value="0.1575" />
+  <!-- Aileron properties -->
+  <!--<xacro:property name="aileron_length" value="0.053" /> --> <!-- [m] -->
+  <!--<xacro:property name="aileron_width" value="0.349" />--> <!-- [m] -->
+  <!--<xacro:property name="aileron_height" value="0.013" /> --> <!-- [m] -->
+  <!--<xacro:property name="aileron_min_angle" value="-0.349066" /> --> <!-- [rad] -->
+  <!--<xacro:property name="aileron_max_angle" value="0.349066" /> --> <!-- [rad] -->
+  <!--<xacro:property name="aileron_color" value="Red" />-->
+  <!-- Component masses -->
+  <!--<xacro:property name="mass_aileron" value="0.1" /> --> <!-- [kg] -->
+  <xacro:property name="mass_flap" value="0.1" /> <!-- [kg] -->
+  <!-- Flap properties -->
+  <xacro:property name="flap_length" value="0.076" /> <!-- [m] -->
+  <xacro:property name="flap_width" value="0.459" /> <!-- [m] -->
+  <xacro:property name="flap_height" value="0.016" /> <!-- [m] -->
+  <xacro:property name="flap_min_angle" value="0.0" /> <!-- [rad] -->
+  <xacro:property name="flap_max_angle" value="1.0" /> <!-- [rad] -->
+  <xacro:property name="flap_color" value="Red" />
+  <xacro:property name="use_mesh" value="true" />
+  <xacro:property name="flap_offset_x" value="0.04" />
+  <xacro:property name="flap_offset_y" value="0.28" />
+  <xacro:property name="flap_offset_z" value="0.02" />
+    <!-- Constants -->
+  <xacro:property name="PI" value="3.1415926535897931" />
   <!-- Property Blocks -->
   <xacro:property name="body_inertia">
     <inertia ixx="0.0347563" ixy="0.0" ixz="0.0" iyy="0.0458929" iyz="0.0" izz="0.0977" /> <!-- [kg m^2] [kg m^2] [kg m^2] [kg m^2] [kg m^2] [kg m^2] -->
   </xacro:property>
+  <xacro:property name="link_inertia">
+    <inertia ixx="0.0347563" ixy="0.0" ixz="0.0" iyy="0.0458929" iyz="0.0" izz="0.0977" /> <!-- [kg m^2] [kg m^2] [kg m^2] [kg m^2] [kg m^2] [kg m^2] -->
+  </xacro:property>
   <!-- inertia of a single rotor, assuming it is a cuboid. Height=3mm, width=15mm -->
   <xacro:property name="rotor_inertia">
     <xacro:box_inertia x="${radius_rotor}" y="0.015" z="0.003" mass="${mass_rotor*rotor_velocity_slowdown_sim}" />
   </xacro:property>
+    <!-- Inertia of the aileron, assuming it is a cuboid -->
+  <xacro:property name="aileron_inertia">
+    <xacro:box_inertia x="${aileron_length}" y="${aileron_width}" z="${aileron_height}" mass="${mass_aileron}" />
+  </xacro:property>
+    <!-- Inertia of the flap, assuming it is a cuboid -->
+  <xacro:property name="flap_inertia">
+    <xacro:box_inertia x="${flap_length}" y="${flap_width}" z="${flap_height}" mass="${mass_flap}" />
+  </xacro:property>
   <!-- Included URDF Files -->
-  <xacro:include filename="$(find spincopter_description)/urdf/multirotor_base.xacro" />
+  <xacro:include filename="$(find spincopter_description)/urdf/rotor_wing_base.xacro" />
   <!-- Instantiate multirotor_base_macro once -->
   <xacro:multirotor_base_macro
@@ -76,5 +110,5 @@
     >
     <origin xyz="${link_offset_base} 0 ${link_offset_top}" rpy="0 ${link_roll} 0" />
-    <xacro:insert_block name="rotor_inertia" />
+    <xacro:insert_block name="link_inertia" />
   </xacro:link_o>
     <xacro:link_o
@@ -84,9 +118,9 @@
     radius_link="${link_radius}"
     length_link="${arm_length}"
-    link_number="1"
+    link_number="2"
     color="Red"
     >
     <origin xyz="-${link_offset_base} 0 ${link_offset_top}" rpy="0 ${link_roll} 0" />
-    <xacro:insert_block name="rotor_inertia" />
+    <xacro:insert_block name="link_inertia" />
   </xacro:link_o>
   <!-- Instantiate rotors -->
@@ -114,5 +148,5 @@
   <xacro:vertical_rotor robot_namespace="${namespace}"
     suffix="back_right"
-    direction="cw"
+    direction="ccw"
     motor_constant="${motor_constant}"
     moment_constant="${moment_constant}"
@@ -132,3 +166,79 @@
     <xacro:insert_block name="rotor_inertia" />
   </xacro:vertical_rotor>
+ <!-- Instantiate the ailerons -->
+ <!--
+  <xacro:control_surface
+    robot_namespace="${namespace}"
+    surface_name="aileron_left"
+    parent="${namespace}/base_link"
+    mass_surface="${mass_aileron}"
+    min_angle="${aileron_min_angle}"
+    max_angle="${aileron_max_angle}"
+    color="${aileron_color}"
+    use_mesh_file="${use_mesh}"
+    mesh_file="package://rotors_description/meshes/techpod/techpod_aileron_left.dae"
+    surface_length="${aileron_length}"
+    surface_width="${aileron_width}"
+    surface_height="${aileron_height}">
+    <axis xyz="0 -1 0" />
+    <origin xyz="0.1095 0.99245 0.115" rpy="0 0 0" />
+    <origin xyz="0 0 0" rpy="0 0 0" />
+    <xacro:insert_block name="aileron_inertia" />
+  </xacro:control_surface>
+  <xacro:control_surface
+    robot_namespace="${namespace}"
+    surface_name="aileron_right"
+    parent="${namespace}/base_link"
+    mass_surface="${mass_aileron}"
+    min_angle="${aileron_min_angle}"
+    max_angle="${aileron_max_angle}"
+    color="${aileron_color}"
+    use_mesh_file="${use_mesh}"
+    mesh_file="package://rotors_description/meshes/techpod/techpod_aileron_right.dae"
+    surface_length="${aileron_length}"
+    surface_width="${aileron_width}"
+    surface_height="${aileron_height}">
+    <axis xyz="0 1 0" />
+    <origin xyz="0.1095 -0.99245 0.115" rpy="0 0 0" />
+    <origin xyz="0 0 0" rpy="0 0 0" />
+    <xacro:insert_block name="aileron_inertia" />
+  </xacro:control_surface>
+-->
+  <!-- Instantiate the flaps -->
+  <xacro:control_surface
+    robot_namespace="${namespace}"
+    surface_name="flap_left"
+    parent="${namespace}/base_link"
+    mass_surface="${mass_flap}"
+    min_angle="${flap_min_angle}"
+    max_angle="${flap_max_angle}"
+    color="${flap_color}"
+    use_mesh_file="${use_mesh}"
+    mesh_file="package://rotors_description/meshes/techpod/techpod_flap_right.dae"
+    surface_length="${flap_length}"
+    surface_width="${flap_width}"
+    surface_height="${flap_height}">
+    <axis xyz="0 -1 0" />   <!-- Joint axis -->
+    <origin xyz="-${flap_offset_x} ${flap_offset_y} ${flap_offset_z}" rpy="0 0 ${PI}" />   <!-- Joint origin -->
+    <origin xyz="0 0 0" rpy="0 0 0" />   <!-- Link origin -->
+    <xacro:insert_block name="flap_inertia" />
+  </xacro:control_surface>
+  <xacro:control_surface
+    robot_namespace="${namespace}"
+    surface_name="flap_right"
+    parent="${namespace}/base_link"
+    mass_surface="${mass_flap}"
+    min_angle="${flap_min_angle}"
+    max_angle="${flap_max_angle}"
+    color="${flap_color}"
+    use_mesh_file="${use_mesh}"
+    mesh_file="package://rotors_description/meshes/techpod/techpod_flap_right.dae"
+    surface_length="${flap_length}"
+    surface_width="${flap_width}"
+    surface_height="${flap_height}">
+    <axis xyz="0 1 0" />   <!-- Joint axis -->
+    <origin xyz="${flap_offset_x} -${flap_offset_y} ${flap_offset_z}" rpy="0 0 0" />
+    <origin xyz="0 0 0" rpy="0 0 0" />   <!-- Link origin -->
+    <xacro:insert_block name="flap_inertia" />
+  </xacro:control_surface>
 </robot>

File: spincopter_description/urdf/spincopter_base.xacro (robot description, xacro)
@@ -19,5 +19,5 @@
   <xacro:include filename="$(find spincopter_description)/urdf/component_snippets.xacro" />
   <!-- Instantiate firefly "mechanics" -->
-  <xacro:include filename="$(find spincopter_description)/urdf/firefly.xacro" />
+  <xacro:include filename="$(find spincopter_description)/urdf/spincopter.xacro" />
   <!-- Instantiate a controller. -->
   <xacro:controller_plugin_macro namespace="${namespace}" imu_sub_topic="imu" />

Commit message: Speed control

File: spincopter_description/urdf/rotor_wing_base.xacro (robot description, xacro)
@@ -71,5 +71,5 @@
     </link>
     <!-- attach multirotor_base_plugin to the base_link -->
-    <gazebo>
+    <!--<gazebo>
       <plugin filename="librotors_gazebo_multirotor_base_plugin.so" name="multirotor_base_plugin">
         <robotNamespace>${robot_namespace}</robotNamespace>
@@ -77,5 +77,5 @@
         <rotorVelocitySlowdownSim>${rotor_velocity_slowdown_sim}</rotorVelocitySlowdownSim>
       </plugin>
-    </gazebo>
+    </gazebo>-->
   </xacro:macro>
   <xacro:macro name="link_o"
@@ -91,8 +91,10 @@
     <link name="${robot_namespace}/link_${link_number}">
       <inertial>
+        <origin xyz="0 0 0" rpy="0 0 0" />
         <mass value="${mass_link}" /> <!-- [kg] -->
         <xacro:insert_block name="inertia" />
       </inertial>
       <visual>
+        <origin xyz="0 0 0" rpy="0 0 0" />
         <geometry>
            <cylinder length="${length_link}" radius="${radius_link}"/>  <!-- [m] -->
@@ -100,4 +102,5 @@
       </visual>
       <collision>
+        <origin xyz="0 0 0" rpy="0 0 0" />
         <geometry>
           <cylinder length="${length_link}" radius="${radius_link}" /> <!-- [m] -->
@@ -173,6 +176,6 @@
     params="robot_namespace surface_name parent mass_surface min_angle
       max_angle color use_mesh_file mesh_file surface_length surface_width
-      surface_height *axis *joint_origin *link_origin *inertia">
-    <joint name="${robot_namespace}/${surface_name}_joint" type="revolute">
+      surface_height surface_x *axis *joint_origin *link_origin *inertia">
+    <joint name="${robot_namespace}/${surface_name}_joint" type= "fixed">  <!--"revolute">-->
       <xacro:insert_block name="joint_origin" />
       <xacro:insert_block name="axis" />
@@ -210,4 +213,43 @@
       </collision>
     </link>
+    <gazebo>
+      <plugin name="${robot_namespace}_${surface_name}" filename="libLiftDragPlugin.so">
+        <robotNamespace>${robot_namespace}</robotNamespace>
+        <a0>0.05984281113</a0>
+        <cla>4.752798721</cla>
+        <cda>0.6417112299</cda>
+        <cma>-1.8</cma>
+        <alpha_stall>0.3391428111</alpha_stall>
+        <cla_stall>-3.85</cla_stall>
+        <cda_stall>-0.9233984055</cda_stall>
+        <cma_stall>0</cma_stall>
+        <cp>-1 2.205 1.5</cp>
+        <area>1.0</area>
+        <air_density>1.2041</air_density>
+        <forward>${surface_x} 0 0</forward>
+        <upward>0 0 1</upward>
+        <control_joint_name>${robot_namespace}/${surface_name}_joint</control_joint_name>
+         <control_joint_rad_to_cl>-2.0</control_joint_rad_to_cl>
+         <!--<link_name>${robot_namespace}/${surface_name}</link_name>-->
+      </plugin>
+ <!--
+      +      <plugin name="rotor_0_blade_1" filename="libLiftDragPlugin.so">
++        <a0>0.1</a0>
++        <alpha_stall>1.4</alpha_stall>
++        <cla>0.2500</cla>
++        <cda>0.10</cda>
++        <cma>0.00</cma>
++        <cla_stall>-0.025</cla_stall>
++        <cda_stall>0.0</cda_stall>
++        <cma_stall>0.0</cma_stall>
++        <area>0.2</area>
++        <air_density>1.2041</air_density>
++        <cp>0.084 0 0</cp>
++        <forward>0 1 0</forward>
++        <upward>0 0 1</upward>
++        <link_name>iris::rotor_0</link_name>
++      </plugin>
+   -->
+    </gazebo>
     <gazebo reference="${robot_namespace}/${surface_name}">
       <material>Gazebo/${color}</material>

File: spincopter_description/urdf/spincopter.xacro (robot description, xacro)
@@ -22,5 +22,5 @@
   <xacro:property name="use_mesh_file" value="False" />
   <xacro:property name="mesh_file" value="package://rotors_description/meshes/firefly.dae" />
-  <xacro:property name="mass" value="1.5" /> <!-- [kg] -->
+  <xacro:property name="mass" value="0.5" /> <!-- [kg] -->
   <xacro:property name="body_width" value="0.1" /> <!-- [m] -->
   <xacro:property name="body_height" value="0.16" /> <!-- [m] -->
@@ -35,31 +35,30 @@
   <xacro:property name="time_constant_down" value="0.025" /> <!-- [s] -->
   <xacro:property name="max_rot_velocity" value="838" /> <!-- [rad/s] -->
-  <xacro:property name="sin30" value="0.5" />
-  <xacro:property name="cos30" value="0.866025403784" />
   <xacro:property name="rotor_drag_coefficient" value="8.06428e-05" />
   <xacro:property name="rolling_moment_coefficient" value="0.000001" />
   <xacro:property name="rotor_roll" value="1.047197" />
   <xacro:property name="link_roll" value="1.57" />
-  <xacro:property name="link_mass" value="0.1" />
+  <xacro:property name="link_mass" value="0.01" />
   <xacro:property name="link_radius" value="0.01" />
   <xacro:property name="link_offset_top" value="0.02" />
   <xacro:property name="link_offset_base" value="0.1575" />
   <!-- Aileron properties -->
-  <!--<xacro:property name="aileron_length" value="0.053" /> --> <!-- [m] -->
-  <!--<xacro:property name="aileron_width" value="0.349" />--> <!-- [m] -->
-  <!--<xacro:property name="aileron_height" value="0.013" /> --> <!-- [m] -->
-  <!--<xacro:property name="aileron_min_angle" value="-0.349066" /> --> <!-- [rad] -->
-  <!--<xacro:property name="aileron_max_angle" value="0.349066" /> --> <!-- [rad] -->
-  <!--<xacro:property name="aileron_color" value="Red" />-->
+  <xacro:property name="aileron_length" value="0.53" />  <!-- [m] -->
+  <xacro:property name="aileron_width" value="0.349" /> <!-- [m] -->
+  <xacro:property name="aileron_height" value="0.013" />  <!-- [m] -->
+  <xacro:property name="aileron_min_angle" value="-0.349066" />  <!-- [rad] -->
+  <xacro:property name="aileron_max_angle" value="0.349066" />  <!-- [rad] -->
+  <xacro:property name="aileron_color" value="Red" />
   <!-- Component masses -->
-  <!--<xacro:property name="mass_aileron" value="0.1" /> --> <!-- [kg] -->
-  <xacro:property name="mass_flap" value="0.1" /> <!-- [kg] -->
+  <xacro:property name="mass_aileron" value="0.1" />  <!-- [kg] -->
+  <xacro:property name="mass_flap" value="0.01" /> <!-- [kg] -->
   <!-- Flap properties -->
-  <xacro:property name="flap_length" value="0.076" /> <!-- [m] -->
-  <xacro:property name="flap_width" value="0.459" /> <!-- [m] -->
-  <xacro:property name="flap_height" value="0.016" /> <!-- [m] -->
+  <xacro:property name="flap_length" value="1" /> <!-- [m] -->
+  <xacro:property name="flap_width" value="0.8" /> <!-- [m] -->
+  <xacro:property name="flap_height" value="0.02" /> <!-- [m] -->
   <xacro:property name="flap_min_angle" value="0.0" /> <!-- [rad] -->
   <xacro:property name="flap_max_angle" value="1.0" /> <!-- [rad] -->
-  <xacro:property name="flap_color" value="Red" />
+  <xacro:property name="flap_color1" value="Red" />
+  <xacro:property name="flap_color2" value="Blue" />
   <xacro:property name="use_mesh" value="true" />
   <xacro:property name="flap_offset_x" value="0.04" />
@@ -70,8 +69,8 @@
   <!-- Property Blocks -->
   <xacro:property name="body_inertia">
-    <inertia ixx="0.0347563" ixy="0.0" ixz="0.0" iyy="0.0458929" iyz="0.0" izz="0.0977" /> <!-- [kg m^2] [kg m^2] [kg m^2] [kg m^2] [kg m^2] [kg m^2] -->
+    <inertia ixx="0.347563" ixy="0.0" ixz="0.0" iyy="0.458929" iyz="0.0" izz="0.977" /> <!-- [kg m^2] [kg m^2] [kg m^2] [kg m^2] [kg m^2] [kg m^2] -->
   </xacro:property>
   <xacro:property name="link_inertia">
-    <inertia ixx="0.0347563" ixy="0.0" ixz="0.0" iyy="0.0458929" iyz="0.0" izz="0.0977" /> <!-- [kg m^2] [kg m^2] [kg m^2] [kg m^2] [kg m^2] [kg m^2] -->
+    <inertia ixx="0.000347563" ixy="0.0" ixz="0.0" iyy="0.000458929" iyz="0.0" izz="0.000977" /> <!-- [kg m^2] [kg m^2] [kg m^2] [kg m^2] [kg m^2] [kg m^2] -->
   </xacro:property>
   <!-- inertia of a single rotor, assuming it is a cuboid. Height=3mm, width=15mm -->
@@ -127,5 +126,5 @@
   <xacro:vertical_rotor
     robot_namespace="${namespace}"
-    suffix="front_left"
+    suffix="left"
     direction="ccw"
     motor_constant="${motor_constant}"
@@ -140,12 +139,13 @@
     rotor_drag_coefficient="${rotor_drag_coefficient}"
     rolling_moment_coefficient="${rolling_moment_coefficient}"
-    color="Red"
+    color="Blue"
     use_own_mesh="False"
     mesh="">
-    <origin xyz="${arm_length} -${rotor_offset_top2} ${rotor_offset_top1}" rpy="${rotor_roll} 0 0" />
+    <origin xyz="${arm_length} ${rotor_offset_top2} ${rotor_offset_top1}" rpy="-${rotor_roll} 0 0" />
     <xacro:insert_block name="rotor_inertia" />
   </xacro:vertical_rotor>
-  <xacro:vertical_rotor robot_namespace="${namespace}"
-    suffix="back_right"
+  <xacro:vertical_rotor
+    robot_namespace="${namespace}"
+    suffix="right"
     direction="ccw"
     motor_constant="${motor_constant}"
@@ -160,12 +160,11 @@
     rotor_drag_coefficient="${rotor_drag_coefficient}"
     rolling_moment_coefficient="${rolling_moment_coefficient}"
-    color="Blue"
+    color="Red"
     use_own_mesh="false"
     mesh="">
-    <origin xyz="-${arm_length} ${rotor_offset_top2} ${rotor_offset_top1}" rpy="-${rotor_roll} 0 0" />
+    <origin xyz="-${arm_length} -${rotor_offset_top2} ${rotor_offset_top1}" rpy="${rotor_roll} 0 0" />
     <xacro:insert_block name="rotor_inertia" />
   </xacro:vertical_rotor>
- <!-- Instantiate the ailerons -->
- <!--
+ <!-- Instantiate the ailerons
   <xacro:control_surface
     robot_namespace="${namespace}"
@@ -213,10 +212,12 @@
     min_angle="${flap_min_angle}"
     max_angle="${flap_max_angle}"
-    color="${flap_color}"
+    color="${flap_color1}"
     use_mesh_file="${use_mesh}"
     mesh_file="package://rotors_description/meshes/techpod/techpod_flap_right.dae"
     surface_length="${flap_length}"
     surface_width="${flap_width}"
-    surface_height="${flap_height}">
+    surface_height="${flap_height}"
+    surface_x="-1"
+    >
     <axis xyz="0 -1 0" />   <!-- Joint axis -->
     <origin xyz="-${flap_offset_x} ${flap_offset_y} ${flap_offset_z}" rpy="0 0 ${PI}" />   <!-- Joint origin -->
@@ -231,10 +232,12 @@
     min_angle="${flap_min_angle}"
     max_angle="${flap_max_angle}"
-    color="${flap_color}"
+    color="${flap_color2}"
     use_mesh_file="${use_mesh}"
     mesh_file="package://rotors_description/meshes/techpod/techpod_flap_right.dae"
     surface_length="${flap_length}"
     surface_width="${flap_width}"
-    surface_height="${flap_height}">
+    surface_height="${flap_height}"
+    surface_x="1"
+    >
     <axis xyz="0 1 0" />   <!-- Joint axis -->
     <origin xyz="${flap_offset_x} -${flap_offset_y} ${flap_offset_z}" rpy="0 0 0" />

File: spincopter_description/urdf/spincopter_base.xacro (robot description, xacro)
@@ -28,4 +28,8 @@
   <!-- Mount an ADIS16448 IMU. -->
   <xacro:default_imu namespace="${namespace}" parent_link="${namespace}/base_link" />
+  <!-- Mount a GPS. -->
+  <xacro:default_gps namespace="${namespace}" parent_link="${namespace}/base_link" />
+  <!-- Mount a magnetometer. -->
+  <xacro:default_magnetometer namespace="${namespace}" parent_link="${namespace}/base_link" />
   <xacro:if value="$(arg enable_ground_truth)">
     <xacro:ground_truth_imu_and_odometry namespace="${namespace}" parent_link="${namespace}/base_link" />
